File: schematics/glove/glove.sch (EAGLE design)
At the start: 21 parts, among them IC1 LM2937

Commit message: 10-19 Prep: Updated Glove and Model schematics and BOMs
Parts:
- JP2, JP3, JP4, JP5, JP6: device EE445L:PINHD-1X3 -> pinhead:PINHD-1X2
Connections:
- net AIN4: now also JP2.1
- net AIN5: now also JP3.1
- net AIN6: now also JP4.1
- net AIN7: now also JP5.1
- net AIN_1: now also JP6.1
- net GND: now also JP2.2, JP3.2, JP4.2, JP5.2, JP6.2
Changed lines of the file:
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@@
 <part name="FRAME1" library="frames" library_urn="urn:adsk.eagle:library:229" deviceset="FRAME_A_L" device="" value="EE445L Lab Board"/>
 <part name="FRAME4" library="frames" library_urn="urn:adsk.eagle:library:229" deviceset="FRAME_A_L" device="" value="EE445L Lab Board"/>
+<part name="JP2" library="pinhead" library_urn="urn:adsk.eagle:library:325" deviceset="PINHD-1X2" device="" package3d_urn="urn:adsk.eagle:package:22435/2"/>
+<part name="JP3" library="pinhead" library_urn="urn:adsk.eagle:library:325" deviceset="PINHD-1X2" device="" package3d_urn="urn:adsk.eagle:package:22435/2"/>
+<part name="JP4" library="pinhead" library_urn="urn:adsk.eagle:library:325" deviceset="PINHD-1X2" device="" package3d_urn="urn:adsk.eagle:package:22435/2"/>
+<part name="JP5" library="pinhead" library_urn="urn:adsk.eagle:library:325" deviceset="PINHD-1X2" device="" package3d_urn="urn:adsk.eagle:package:22435/2"/>
+<part name="JP6" library="pinhead" library_urn="urn:adsk.eagle:library:325" deviceset="PINHD-1X2" device="" package3d_urn="urn:adsk.eagle:package:22435/2"/>
 <part name="SUPPLY1" library="EE445L" deviceset="GND" device=""/>
 <part name="SUPPLY2" library="EE445L" deviceset="GND" device=""/>
@@
 <part name="SUPPLY5" library="EE445L" deviceset="GND" device=""/>
 <part name="SUPPLY8" library="EE445L" deviceset="GND" device=""/>
-<part name="JP2" library="EE445L" deviceset="PINHD-1X3" device=""/>
-<part name="JP3" library="EE445L" deviceset="PINHD-1X3" device=""/>
-<part name="JP4" library="EE445L" deviceset="PINHD-1X3" device=""/>
-<part name="JP5" library="EE445L" deviceset="PINHD-1X3" device=""/>
-<part name="JP6" library="EE445L" deviceset="PINHD-1X3" device=""/>
 </parts>
 <sheets>
@@
 <attribute name="DRAWING_NAME" x="477.52" y="240.03" size="2.54" layer="94"/>
 </instance>
+<instance part="JP2" gate="G$1" x="411.48" y="337.82" smashed="yes">
+<attribute name="NAME" x="405.13" y="343.535" size="1.778" layer="95"/>
+<attribute name="VALUE" x="405.13" y="332.74" size="1.778" layer="96"/>
+</instance>
+<instance part="JP3" gate="G$1" x="411.48" y="325.12" smashed="yes">
+<attribute name="NAME" x="405.13" y="330.835" size="1.778" layer="95"/>
+<attribute name="VALUE" x="405.13" y="320.04" size="1.778" layer="96"/>
+</instance>
+<instance part="JP4" gate="G$1" x="411.48" y="312.42" smashed="yes">
+<attribute name="NAME" x="405.13" y="318.135" size="1.778" layer="95"/>
+<attribute name="VALUE" x="405.13" y="307.34" size="1.778" layer="96"/>
+</instance>
+<instance part="JP5" gate="G$1" x="411.48" y="299.72" smashed="yes">
+<attribute name="NAME" x="405.13" y="305.435" size="1.778" layer="95"/>
+<attribute name="VALUE" x="405.13" y="294.64" size="1.778" layer="96"/>
+</instance>
+<instance part="JP6" gate="G$1" x="411.48" y="287.02" smashed="yes">
+<attribute name="NAME" x="405.13" y="292.735" size="1.778" layer="95"/>
+<attribute name="VALUE" x="405.13" y="281.94" size="1.778" layer="96"/>
+</instance>
 <instance part="SUPPLY1" gate="GND" x="421.64" y="337.82" smashed="yes" rot="R90">
 <attribute name="VALUE" x="426.339" y="333.375" size="1.778" layer="96" rot="R90"/>
@@
 <instance part="SUPPLY8" gate="GND" x="421.64" y="287.02" smashed="yes" rot="R90">
 <attribute name="VALUE" x="426.339" y="282.575" size="1.778" layer="96" rot="R90"/>
-</instance>
-<instance part="JP2" gate="A" x="408.94" y="337.82" smashed="yes">
-<attribute name="NAME" x="402.59" y="343.535" size="1.778" layer="95"/>
-<attribute name="VALUE" x="402.59" y="330.2" size="1.778" layer="96"/>
-</instance>
-<instance part="JP3" gate="A" x="408.94" y="322.58" smashed="yes">
-<attribute name="NAME" x="402.59" y="328.295" size="1.778" layer="95"/>
-<attribute name="VALUE" x="402.59" y="314.96" size="1.778" layer="96"/>
-</instance>
-<instance part="JP4" gate="A" x="408.94" y="307.34" smashed="yes">
-<attribute name="NAME" x="402.59" y="313.055" size="1.778" layer="95"/>
-<attribute name="VALUE" x="402.59" y="299.72" size="1.778" layer="96"/>
-</instance>
-<instance part="JP5" gate="A" x="408.94" y="292.1" smashed="yes">
-<attribute name="NAME" x="402.59" y="297.815" size="1.778" layer="95"/>
-<attribute name="VALUE" x="402.59" y="284.48" size="1.778" layer="96"/>
-</instance>
-<instance part="JP6" gate="A" x="408.94" y="274.32" smashed="yes">
-<attribute name="NAME" x="402.59" y="280.035" size="1.778" layer="95"/>
-<attribute name="VALUE" x="402.59" y="266.7" size="1.778" layer="96"/>
 </instance>
 </instances>
@@
 <wire x1="147.32" y1="368.3" x2="147.32" y2="365.76" width="0.1524" layer="91"/>
 </segment>
+<segment>
+<pinref part="JP2" gate="G$1" pin="2"/>
+<pinref part="SUPPLY1" gate="GND" pin="GND"/>
+<wire x1="408.94" y1="337.82" x2="419.1" y2="337.82" width="0.1524" layer="91"/>
+</segment>
+<segment>
+<pinref part="JP3" gate="G$1" pin="2"/>
+<pinref part="SUPPLY2" gate="GND" pin="GND"/>
+<wire x1="408.94" y1="325.12" x2="419.1" y2="325.12" width="0.1524" layer="91"/>
+</segment>
+<segment>
+<pinref part="JP4" gate="G$1" pin="2"/>
+<pinref part="SUPPLY4" gate="GND" pin="GND"/>
+<wire x1="408.94" y1="312.42" x2="419.1" y2="312.42" width="0.1524" layer="91"/>
+</segment>
+<segment>
+<pinref part="JP5" gate="G$1" pin="2"/>
+<pinref part="SUPPLY5" gate="GND" pin="GND"/>
+<wire x1="408.94" y1="299.72" x2="419.1" y2="299.72" width="0.1524" layer="91"/>
+</segment>
+<segment>
+<pinref part="JP6" gate="G$1" pin="2"/>
+<pinref part="SUPPLY8" gate="GND" pin="GND"/>
+<wire x1="408.94" y1="287.02" x2="419.1" y2="287.02" width="0.1524" layer="91"/>
+</segment>
 </net>
 <net name="+3V3" class="0">
@@
 <label x="147.32" y="149.86" size="1.778" layer="95"/>
 </segment>
+<segment>
+<pinref part="JP6" gate="G$1" pin="1"/>
+<wire x1="408.94" y1="289.56" x2="396.24" y2="289.56" width="0.1524" layer="91"/>
+<label x="396.24" y="289.56" size="1.778" layer="95"/>
+</segment>
 </net>
 <net name="RSTB_8266" class="0">
@@
 <segment>
 <pinref part="U$2" gate="G$4" pin="PD3"/>
-<wire x1="345.44" y1="317.5" x2="370.84" y2="317.5" width="0.1524" layer="91"/>
+<wire x1="345.44" y1="317.5" x2="391.16" y2="317.5" width="0.1524" layer="91"/>
 <label x="355.6" y="317.5" size="1.778" layer="95"/>
+<wire x1="391.16" y1="317.5" x2="391.16" y2="340.36" width="0.1524" layer="91"/>
+<pinref part="JP2" gate="G$1" pin="1"/>
+<wire x1="391.16" y1="340.36" x2="408.94" y2="340.36" width="0.1524" layer="91"/>
 </segment>
 </net>
@@
 <segment>
 <pinref part="U$2" gate="G$4" pin="PD2"/>
-<wire x1="345.44" y1="314.96" x2="370.84" y2="314.96" width="0.1524" layer="91"/>
+<wire x1="345.44" y1="314.96" x2="393.7" y2="314.96" width="0.1524" layer="91"/>
 <label x="355.6" y="314.96" size="1.778" layer="95"/>
+<wire x1="393.7" y1="314.96" x2="393.7" y2="327.66" width="0.1524" layer="91"/>
+<pinref part="JP3" gate="G$1" pin="1"/>
+<wire x1="393.7" y1="327.66" x2="408.94" y2="327.66" width="0.1524" layer="91"/>
 </segment>
 </net>
@@
 <pinref part="U$2" gate="G$4" pin="PD1"/>
 <label x="355.6" y="312.42" size="1.778" layer="95"/>
-<wire x1="345.44" y1="312.42" x2="370.84" y2="312.42" width="0.1524" layer="91"/>
+<wire x1="345.44" y1="312.42" x2="396.24" y2="312.42" width="0.1524" layer="91"/>
+<pinref part="JP4" gate="G$1" pin="1"/>
+<wire x1="396.24" y1="312.42" x2="396.24" y2="314.96" width="0.1524" layer="91"/>
+<wire x1="396.24" y1="314.96" x2="408.94" y2="314.96" width="0.1524" layer="91"/>
 </segment>
 </net>
@@
 <pinref part="U$2" gate="G$4" pin="PD0"/>
 <label x="355.6" y="309.88" size="1.778" layer="95"/>
-<wire x1="345.44" y1="309.88" x2="370.84" y2="309.88" width="0.1524" layer="91"/>
+<wire x1="345.44" y1="309.88" x2="396.24" y2="309.88" width="0.1524" layer="91"/>
+<pinref part="JP5" gate="G$1" pin="1"/>
+<wire x1="396.24" y1="309.88" x2="396.24" y2="302.26" width="0.1524" layer="91"/>
+<wire x1="396.24" y1="302.26" x2="408.94" y2="302.26" width="0.1524" layer="91"/>
 </segment>
 </net>
@@
 will not be understood (or retained) with this version.
 </note>
+<note version="8.3" severity="warning">
+Since Version 8.3, EAGLE supports the association of 3D packages
+with devices in libraries, schematics, and board files. Those 3D
+packages will not be understood (or retained) with this version.
+</note>
 <note version="8.4" severity="warning">
