File: schematics/model/model.brd (EAGLE design)
At the start: 114.3 x 114 mm, 16 parts, among them IC1 LM2937

Commit message: 10-19 Prep: Updated Glove and Model schematics and BOMs
Parts:
- added JP2, JP3, JP4, JP5, JP6: (no value), EE445L:1X03
Connections:
- net PD2 renamed AIN5
- net SSI1_FS renamed AIN6
- net SSI1_MOSI renamed AIN4
- net SSI_SCK renamed AIN7
- removed net PB5: U$2.J1-2
- removed net PB7: U$2.J2-15
- removed net PC4: U$2.J4-37
- removed net TACH: U$2.J1-7
- new net PWM1: JP3.2, U$2.J2-15
- new net PWM2: JP4.2, U$2.J1-7
- new net PWM3: JP5.2, U$2.J1-2
- new net PWM6: JP6.2, U$2.J4-37
- net +5V: now also JP2.1, JP3.1, JP4.1, JP5.1, JP6.1
- net GND: now also JP2.3, JP3.3, JP4.3, JP5.3, JP6.3
- net PWM0: now also JP2.2
Routing:
- net PWM3: track 0.00 -> 149.7 mm, vias 0 -> 2
- net PWM2: track 0.00 -> 131.6 mm, vias 0 -> 4
- net +5V: track 67.7 -> 169.5 mm, vias 0 -> 1
- net PWM6: track 0.00 -> 38.2 mm, vias 0 -> 1
- net GND: track 215.1 -> 253.2 mm
- net PWM0: track 0.00 -> 32.2 mm
- net PWM1: track 0.00 -> 30.4 mm, vias 0 -> 1
- net 8266_TX: track 64.1 -> 63.4 mm, vias 0 -> 1
Changed lines of the file:
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@@
 <drawing>
 <settings>
-<setting alwaysvectorfont="yes"/>
+<setting alwaysvectorfont="no"/>
 <setting verticaltext="up"/>
 </settings>
@@
 <attribute name="VALUE" x="80.645" y="91.059" size="1.27" layer="27" ratio="10"/>
 </element>
+<element name="JP2" library="EE445L" package="1X03" value="" x="97.79" y="50.8" smashed="yes" rot="R180">
+<attribute name="NAME" x="101.6762" y="48.9712" size="1.27" layer="25" ratio="10" rot="R180"/>
+<attribute name="VALUE" x="101.6" y="53.975" size="1.27" layer="27" rot="R180"/>
+</element>
+<element name="JP3" library="EE445L" package="1X03" value="" x="97.79" y="55.88" smashed="yes" rot="R180">
+<attribute name="NAME" x="101.6762" y="54.0512" size="1.27" layer="25" ratio="10" rot="R180"/>
+<attribute name="VALUE" x="101.6" y="59.055" size="1.27" layer="27" rot="R180"/>
+</element>
+<element name="JP4" library="EE445L" package="1X03" value="" x="97.79" y="60.96" smashed="yes" rot="R180">
+<attribute name="NAME" x="101.6762" y="59.1312" size="1.27" layer="25" ratio="10" rot="R180"/>
+<attribute name="VALUE" x="101.6" y="64.135" size="1.27" layer="27" rot="R180"/>
+</element>
+<element name="JP5" library="EE445L" package="1X03" value="" x="97.79" y="66.04" smashed="yes" rot="R180">
+<attribute name="NAME" x="101.6762" y="64.2112" size="1.27" layer="25" ratio="10" rot="R180"/>
+<attribute name="VALUE" x="101.6" y="69.215" size="1.27" layer="27" rot="R180"/>
+</element>
+<element name="JP6" library="EE445L" package="1X03" value="" x="97.79" y="71.12" smashed="yes" rot="R180">
+<attribute name="NAME" x="101.6762" y="69.2912" size="1.27" layer="25" ratio="10" rot="R180"/>
+<attribute name="VALUE" x="101.6" y="74.295" size="1.27" layer="27" rot="R180"/>
+</element>
 </elements>
 <signals>
@@
 <wire x1="77.47" y1="77.47" x2="76.2" y2="78.74" width="0.1524" layer="1"/>
 <wire x1="76.2" y1="78.74" x2="73.66" y2="78.74" width="0.1524" layer="1"/>
+<contactref element="JP2" pad="3"/>
+<contactref element="JP3" pad="3"/>
+<contactref element="JP4" pad="3"/>
+<contactref element="JP5" pad="3"/>
+<contactref element="JP6" pad="3"/>
+<wire x1="95.25" y1="71.12" x2="95.25" y2="66.04" width="0.1524" layer="1"/>
+<wire x1="95.25" y1="60.96" x2="95.25" y2="66.04" width="0.1524" layer="1"/>
+<wire x1="95.25" y1="60.96" x2="95.25" y2="55.88" width="0.1524" layer="1"/>
+<wire x1="95.25" y1="55.88" x2="95.25" y2="50.8" width="0.1524" layer="1"/>
+<wire x1="95.25" y1="71.12" x2="77.47" y2="71.12" width="0.1524" layer="1"/>
 </signal>
 <signal name="+3V3">
@@
 <wire x1="29.21" y1="67.31" x2="31.75" y2="67.31" width="0.1524" layer="16"/>
 <wire x1="31.75" y1="67.31" x2="33.02" y2="66.04" width="0.1524" layer="16"/>
-<wire x1="33.02" y1="33.02" x2="34.29" y2="31.75" width="0.1524" layer="16"/>
-<wire x1="34.29" y1="31.75" x2="50.8" y2="31.75" width="0.1524" layer="16"/>
-<wire x1="50.8" y1="31.75" x2="54.61" y2="27.94" width="0.1524" layer="16"/>
-<wire x1="54.61" y1="27.94" x2="54.61" y2="26.67" width="0.1524" layer="16"/>
-<wire x1="33.02" y1="66.04" x2="33.02" y2="33.02" width="0.1524" layer="16"/>
+<wire x1="33.02" y1="66.04" x2="33.02" y2="62.23" width="0.1524" layer="16"/>
+<via x="33.02" y="62.23" extent="1-16" drill="0.35"/>
+<wire x1="33.02" y1="62.23" x2="33.02" y2="33.02" width="0.1524" layer="1"/>
+<wire x1="33.02" y1="33.02" x2="34.29" y2="31.75" width="0.1524" layer="1"/>
+<wire x1="34.29" y1="31.75" x2="49.53" y2="31.75" width="0.1524" layer="1"/>
+<wire x1="49.53" y1="31.75" x2="54.61" y2="26.67" width="0.1524" layer="1"/>
 </signal>
 <signal name="RSTB_8266">
@@
 <contactref element="U$2" pad="J4-38"/>
 </signal>
-<signal name="TACH">
+<signal name="PWM2">
 <contactref element="U$2" pad="J1-7"/>
-</signal>
-<signal name="PB5">
+<contactref element="JP4" pad="2"/>
+<wire x1="27.94" y1="63.5" x2="22.86" y2="58.42" width="0.1524" layer="16"/>
+<wire x1="22.86" y1="58.42" x2="22.86" y2="35.56" width="0.1524" layer="16"/>
+<wire x1="22.86" y1="35.56" x2="24.13" y2="34.29" width="0.1524" layer="16"/>
+<wire x1="24.13" y1="34.29" x2="54.61" y2="34.29" width="0.1524" layer="16"/>
+<via x="54.61" y="34.29" extent="1-16" drill="0.35"/>
+<wire x1="54.61" y1="34.29" x2="73.66" y2="34.29" width="0.1524" layer="1"/>
+<wire x1="73.66" y1="34.29" x2="81.28" y2="41.91" width="0.1524" layer="1"/>
+<wire x1="81.28" y1="41.91" x2="81.28" y2="43.18" width="0.1524" layer="1"/>
+<via x="81.28" y="43.18" extent="1-16" drill="0.35"/>
+<wire x1="81.28" y1="43.18" x2="81.28" y2="62.23" width="0.1524" layer="16"/>
+<via x="81.28" y="62.23" extent="1-16" drill="0.35"/>
+<wire x1="81.28" y1="62.23" x2="86.36" y2="62.23" width="0.1524" layer="1"/>
+<wire x1="86.36" y1="62.23" x2="90.17" y2="58.42" width="0.1524" layer="1"/>
+<via x="90.17" y="58.42" extent="1-16" drill="0.35"/>
+<wire x1="90.17" y1="58.42" x2="95.25" y2="58.42" width="0.1524" layer="16"/>
+<wire x1="95.25" y1="58.42" x2="97.79" y2="60.96" width="0.1524" layer="16"/>
+</signal>
+<signal name="PWM3">
 <contactref element="U$2" pad="J1-2"/>
+<contactref element="JP5" pad="2"/>
+<wire x1="27.94" y1="76.2" x2="21.59" y2="69.85" width="0.1524" layer="16"/>
+<wire x1="21.59" y1="69.85" x2="21.59" y2="35.56" width="0.1524" layer="16"/>
+<wire x1="21.59" y1="35.56" x2="26.67" y2="30.48" width="0.1524" layer="16"/>
+<wire x1="26.67" y1="30.48" x2="54.61" y2="30.48" width="0.1524" layer="16"/>
+<via x="54.61" y="30.48" extent="1-16" drill="0.35"/>
+<wire x1="54.61" y1="30.48" x2="72.39" y2="30.48" width="0.1524" layer="1"/>
+<wire x1="83.82" y1="41.91" x2="72.39" y2="30.48" width="0.1524" layer="1"/>
+<wire x1="83.82" y1="41.91" x2="83.82" y2="43.18" width="0.1524" layer="1"/>
+<via x="83.82" y="43.18" extent="1-16" drill="0.35"/>
+<wire x1="83.82" y1="63.5" x2="83.82" y2="43.18" width="0.1524" layer="16"/>
+<wire x1="83.82" y1="63.5" x2="96.52" y2="63.5" width="0.1524" layer="16"/>
+<wire x1="96.52" y1="63.5" x2="97.79" y2="64.77" width="0.1524" layer="16"/>
+<wire x1="97.79" y1="64.77" x2="97.79" y2="66.04" width="0.1524" layer="16"/>
 </signal>
 <signal name="PWM0">
 <contactref element="U$2" pad="J2-14"/>
-</signal>
-<signal name="PB7">
+<contactref element="JP2" pad="2"/>
+<wire x1="97.79" y1="50.8" x2="95.25" y2="48.26" width="0.1524" layer="1"/>
+<wire x1="95.25" y1="48.26" x2="87.63" y2="48.26" width="0.1524" layer="1"/>
+<wire x1="74.6426" y1="61.2474" x2="74.6426" y2="61.36700625" width="0.1524" layer="1"/>
+<wire x1="73.66" y1="62.34960625" x2="73.66" y2="63.5" width="0.1524" layer="1"/>
+<wire x1="74.6426" y1="61.36700625" x2="73.66" y2="62.34960625" width="0.1524" layer="1"/>
+<wire x1="87.63" y1="48.26" x2="74.6426" y2="61.2474" width="0.1524" layer="1"/>
+</signal>
+<signal name="PWM1">
 <contactref element="U$2" pad="J2-15"/>
+<contactref element="JP3" pad="2"/>
+<wire x1="97.79" y1="55.88" x2="95.25" y2="53.34" width="0.1524" layer="16"/>
+<wire x1="95.25" y1="53.34" x2="87.63" y2="53.34" width="0.1524" layer="16"/>
+<via x="87.63" y="53.34" extent="1-16" drill="0.35"/>
+<wire x1="87.63" y1="53.34" x2="74.93" y2="66.04" width="0.1524" layer="1"/>
+<wire x1="74.93" y1="66.04" x2="73.66" y2="66.04" width="0.1524" layer="1"/>
 </signal>
 <signal name="+5V">
@@
 <wire x1="30.48" y1="80.01" x2="30.48" y2="78.74" width="0.1524" layer="1"/>
 <wire x1="26.67" y1="74.93" x2="26.67" y2="80.01" width="0.1524" layer="1"/>
+<contactref element="JP2" pad="1"/>
+<contactref element="JP3" pad="1"/>
+<contactref element="JP4" pad="1"/>
+<contactref element="JP5" pad="1"/>
+<contactref element="JP6" pad="1"/>
+<wire x1="100.33" y1="50.8" x2="100.33" y2="55.88" width="0.1524" layer="1"/>
+<wire x1="100.33" y1="55.88" x2="100.33" y2="60.96" width="0.1524" layer="1"/>
+<wire x1="100.33" y1="60.96" x2="100.33" y2="66.04" width="0.1524" layer="1"/>
+<wire x1="100.33" y1="66.04" x2="100.33" y2="71.12" width="0.1524" layer="1"/>
+<wire x1="100.33" y1="71.12" x2="100.33" y2="74.93" width="0.1524" layer="1"/>
+<wire x1="88.9" y1="86.36" x2="82.55" y2="86.36" width="0.1524" layer="1"/>
+<via x="82.55" y="86.36" extent="1-16" drill="0.35"/>
+<wire x1="82.55" y1="86.36" x2="38.1" y2="86.36" width="0.1524" layer="16"/>
+<wire x1="38.1" y1="86.36" x2="30.48" y2="78.74" width="0.1524" layer="16"/>
+<wire x1="100.33" y1="74.93" x2="88.9" y2="86.36" width="0.1524" layer="1"/>
 </signal>
 <signal name="RESET">
@@
 <contactref element="U$2" pad="J4-33"/>
 </signal>
-<signal name="SSI1_MOSI">
+<signal name="AIN4">
 <contactref element="U$2" pad="J3-26"/>
 </signal>
-<signal name="PD2">
+<signal name="AIN5">
 <contactref element="U$2" pad="J3-25"/>
 </signal>
-<signal name="SSI1_FS">
+<signal name="AIN6">
 <contactref element="U$2" pad="J3-24"/>
 </signal>
-<signal name="SSI_SCK">
+<signal name="AIN7">
 <contactref element="U$2" pad="J3-23"/>
 </signal>
@@
 <contactref element="U$2" pad="J4-36"/>
 </signal>
-<signal name="PC4">
+<signal name="PWM6">
 <contactref element="U$2" pad="J4-37"/>
+<contactref element="JP6" pad="2"/>
+<wire x1="97.79" y1="71.12" x2="93.98" y2="74.93" width="0.1524" layer="1"/>
+<wire x1="93.98" y1="74.93" x2="78.74" y2="74.93" width="0.1524" layer="1"/>
+<via x="78.74" y="74.93" extent="1-16" drill="0.35"/>
+<wire x1="78.74" y1="74.93" x2="68.58" y2="74.93" width="0.1524" layer="16"/>
+<wire x1="68.58" y1="74.93" x2="67.31" y2="73.66" width="0.1524" layer="16"/>
+<wire x1="67.31" y1="73.66" x2="67.31" y2="72.39" width="0.1524" layer="16"/>
+<wire x1="67.31" y1="72.39" x2="68.58" y2="71.12" width="0.1524" layer="16"/>
+<wire x1="68.58" y1="71.12" x2="71.12" y2="71.12" width="0.1524" layer="16"/>
 </signal>
 <signal name="PB0">

Commit message: Submitted PCB
Parts:
- removed C1: 4.7uf, EE445L:CAP200MILPOLARIZED
- removed C19: 0.1uf, EE445L:CAP200MIL
- removed U$1: ESP_8266, EE445L:ESP8266
- moved JP1 41.3 mm to (44.5, 45.7)
- moved 3.3V 41.3 mm to (47.0, 68.6)
- moved 5.0V 41.3 mm to (47.0, 73.7)
- moved C3 41.3 mm to (38.1, 53.3)
- moved GND 41.3 mm to (47.0, 63.5)
- moved IC1 41.3 mm to (38.1, 67.3)
- moved U$6 41.3 mm to (49.5, 50.8)
- moved U$5 41.3 mm to (48.3, 55.9)
- moved C5 7.73 mm to (95.2, 105.4)
- moved LED2 7.73 mm to (86.4, 91.4)
- moved R1 7.73 mm to (87.6, 100.3)
- moved R3 7.73 mm to (101.6, 97.8)
Connections:
- net +3V3: no longer C1.+, C19.2, R3.2, U$1.CH_EN, U$1.VDD
- net 8266_GPIO_0: no longer U$1.GPIO_0
- net 8266_GPIO_2: no longer U$1.GPIO_2
- net 8266_RX: no longer U$1.RXD
- net 8266_TX: no longer U$1.TXD
- net GND: no longer C1.-, C19.1, U$1.GND
- net RSTB_8266: no longer U$1.RST_B
Routing:
- net +5V: track 169.5 -> 208.1 mm
- net +3V3: track 214.9 -> 185.9 mm
- net PWM3: track 149.7 -> 129.6 mm
- net 8266_RX: track 57.5 -> 46.1 mm
- net 8266_TX: track 63.4 -> 56.2 mm
- net GND: track 253.2 -> 257.1 mm
- net 8266_GPIO_2: track 70.4 -> 68.6 mm
- net RSTB_8266: track 52.2 -> 50.9 mm
- net 8266_GPIO_0: track 96.2 -> 96.7 mm
