File: schematics/model/model.sch (EAGLE design)
At the start: 16 parts, among them IC1 LM2937

Commit message: 10-19 Prep: Updated Glove and Model schematics and BOMs
Parts:
- added JP2, JP3, JP4, JP5, JP6: (no value), EE445L:PINHD-1X3
Connections:
- net PD2 renamed AIN5
- net SSI1_FS renamed AIN6
- net SSI1_MOSI renamed AIN4
- net SSI_SCK renamed AIN7
- removed net PB5: U$2G$2.PB5
- removed net PB7: U$2G$2.PB7
- removed net PC4: U$2G$3.PC4
- removed net TACH: U$2G$2.PB4
- new net PWM1: JP3.2, U$2G$2.PB7
- new net PWM2: JP4.2, U$2G$2.PB4
- new net PWM3: JP5.2, U$2G$2.PB5
- new net PWM6: JP6.2, U$2G$3.PC4
- net +5V: now also JP2.1, JP3.1, JP4.1, JP5.1, JP6.1
- net GND: now also JP2.3, JP3.3, JP4.3, JP5.3, JP6.3
- net PWM0: now also JP2.2
Other:
- note added: "Pin Headers for 5 Flex Sensors"

Commit message: Submitted PCB
Parts:
- removed C1: 4.7uf, EE445L:CAPACITOR_POLARIZEDE5-6
- removed C19: 0.1uf, EE445L:CAPACITOR050-024X044
- removed U$1: ESP_8266, EE445L:ESP_8266
Connections:
- net +3V3: no longer C1.+, C19.2, R3.2, U$1.4-CH_EN, U$1.8-VDD
- net 8266_GPIO_0: no longer U$1.5-GPIO_0
- net 8266_GPIO_2: no longer U$1.3-GPIO_2
- net 8266_RX: no longer U$1.7-RXD
- net 8266_TX: no longer U$1.2-TXD
- net GND: no longer C1.-, C19.1, U$1.1-GND
- net RSTB_8266: no longer U$1.6-RST_B
Other:
- note removed: "WiFi Block"
Changed lines of the file:
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@@
 <parts>
 <part name="R3" library="EE445L" deviceset="RESISTOR" device="0204/7" value="10K"/>
-<part name="C1" library="EE445L" deviceset="CAPACITOR_POLARIZED" device="E5-6" value="4.7uf"/>
-<part name="C19" library="EE445L" deviceset="CAPACITOR" device="050-024X044" value="0.1uf"/>
-<part name="SUPPLY3" library="EE445L" deviceset="GND" device=""/>
-<part name="SUPPLY32" library="EE445L" deviceset="GND" device=""/>
-<part name="SUPPLY35" library="EE445L" deviceset="GND" device=""/>
-<part name="U$1" library="EE445L" deviceset="ESP_8266" device=""/>
 <part name="5.0V" library="EE445L" deviceset="TP_LOOP" device=""/>
 <part name="U$2" library="EE445L" deviceset="TM4C_BP" device=""/>
@@
 <part name="SUPPLY7" library="EE445L" deviceset="GND" device=""/>
 <part name="LED2" library="EE445L" deviceset="LED" device="3MM"/>
-<part name="+3V4" library="EE445L" deviceset="+3V3" device=""/>
 <part name="FRAME2" library="frames" library_urn="urn:adsk.eagle:library:229" deviceset="FRAME_A_L" device="" value="EE445L Lab Board"/>
 <part name="FRAME1" library="frames" library_urn="urn:adsk.eagle:library:229" deviceset="FRAME_A_L" device="" value="EE445L Lab Board"/>
@@
 <sheet>
 <plain>
-<text x="228.854" y="130.302" size="5.08" layer="97">WiFi Block</text>
 <text x="58.42" y="403.86" size="1.778" layer="91">Use this jumper to
 measure current</text>
@@
 <attribute name="VALUE" x="178.562" y="173.99" size="1.778" layer="96" rot="R90"/>
 </instance>
-<instance part="C1" gate="G$1" x="238.76" y="160.02" smashed="yes">
-<attribute name="NAME" x="239.776" y="160.655" size="1.778" layer="95"/>
-<attribute name="VALUE" x="232.156" y="155.829" size="1.778" layer="96"/>
-</instance>
-<instance part="C19" gate="G$1" x="251.46" y="157.48" smashed="yes" rot="R180">
-<attribute name="NAME" x="252.984" y="159.385" size="1.778" layer="95"/>
-<attribute name="VALUE" x="245.364" y="154.051" size="1.778" layer="96"/>
-</instance>
-<instance part="SUPPLY3" gate="GND" x="218.44" y="132.08" smashed="yes">
-<attribute name="VALUE" x="211.455" y="132.461" size="1.778" layer="96"/>
-</instance>
-<instance part="SUPPLY32" gate="GND" x="238.76" y="144.78" smashed="yes">
-<attribute name="VALUE" x="231.775" y="145.161" size="1.778" layer="96"/>
-</instance>
-<instance part="SUPPLY35" gate="GND" x="251.46" y="144.78" smashed="yes">
-<attribute name="VALUE" x="244.475" y="145.161" size="1.778" layer="96"/>
-</instance>
-<instance part="U$1" gate="G$1" x="213.36" y="157.48" smashed="yes"/>
 <instance part="5.0V" gate="G$1" x="93.98" y="401.32" smashed="yes">
 <attribute name="NAME" x="91.44" y="404.368" size="1.778" layer="95"/>
@@
 <attribute name="VALUE" x="153.035" y="368.808" size="1.778" layer="96" rot="R90"/>
 </instance>
-<instance part="+3V4" gate="G$1" x="203.2" y="193.04" smashed="yes">
-<attribute name="VALUE" x="210.82" y="193.04" size="1.778" layer="96" rot="R180"/>
-</instance>
 <instance part="FRAME2" gate="G$1" x="287.02" y="0" smashed="yes"/>
 <instance part="FRAME2" gate="G$2" x="459.74" y="0" smashed="yes">
@@
 <nets>
 <net name="GND" class="0">
-<segment>
-<pinref part="SUPPLY32" gate="GND" pin="GND"/>
-<pinref part="C1" gate="G$1" pin="-"/>
-<wire x1="238.76" y1="147.32" x2="238.76" y2="154.94" width="0.1524" layer="91"/>
-</segment>
-<segment>
-<pinref part="C19" gate="G$1" pin="1"/>
-<pinref part="SUPPLY35" gate="GND" pin="GND"/>
-<wire x1="251.46" y1="154.94" x2="251.46" y2="147.32" width="0.1524" layer="91"/>
-</segment>
-<segment>
-<pinref part="SUPPLY3" gate="GND" pin="GND"/>
-<wire x1="218.44" y1="137.16" x2="218.44" y2="134.62" width="0.1524" layer="91"/>
-<pinref part="U$1" gate="G$1" pin="1-GND"/>
-</segment>
 <segment>
 <pinref part="U$2" gate="G$7" pin="GND2"/>
@@
 <pinref part="R1" gate="G$1" pin="2"/>
 </segment>
-<segment>
-<pinref part="R3" gate="G$1" pin="2"/>
-<pinref part="C1" gate="G$1" pin="+"/>
-<wire x1="238.76" y1="162.56" x2="238.76" y2="182.88" width="0.1524" layer="91"/>
-<wire x1="238.76" y1="182.88" x2="218.44" y2="182.88" width="0.1524" layer="91"/>
-<wire x1="218.44" y1="182.88" x2="218.44" y2="177.8" width="0.1524" layer="91"/>
-<pinref part="C19" gate="G$1" pin="2"/>
-<wire x1="251.46" y1="162.56" x2="251.46" y2="182.88" width="0.1524" layer="91"/>
-<wire x1="251.46" y1="182.88" x2="238.76" y2="182.88" width="0.1524" layer="91"/>
-<junction x="238.76" y="182.88"/>
-<wire x1="198.12" y1="160.02" x2="190.5" y2="160.02" width="0.1524" layer="91"/>
-<wire x1="190.5" y1="160.02" x2="190.5" y2="182.88" width="0.1524" layer="91"/>
-<wire x1="190.5" y1="182.88" x2="203.2" y2="182.88" width="0.1524" layer="91"/>
-<junction x="218.44" y="182.88"/>
-<pinref part="U$1" gate="G$1" pin="4-CH_EN"/>
-<pinref part="U$1" gate="G$1" pin="8-VDD"/>
-<wire x1="203.2" y1="182.88" x2="218.44" y2="182.88" width="0.1524" layer="91"/>
-<wire x1="175.26" y1="182.88" x2="190.5" y2="182.88" width="0.1524" layer="91"/>
-<junction x="190.5" y="182.88"/>
-<pinref part="+3V4" gate="G$1" pin="+3V3"/>
-<wire x1="203.2" y1="190.5" x2="203.2" y2="182.88" width="0.1524" layer="91"/>
-<junction x="203.2" y="182.88"/>
-</segment>
 </net>
 <net name="8266_RX" class="0">
 <segment>
-<wire x1="198.12" y1="144.78" x2="172.72" y2="144.78" width="0.1524" layer="91"/>
 <wire x1="172.72" y1="144.78" x2="172.72" y2="157.48" width="0.1524" layer="91"/>
 <wire x1="172.72" y1="157.48" x2="127" y2="157.48" width="0.1524" layer="91"/>
-<pinref part="U$1" gate="G$1" pin="7-RXD"/>
 <pinref part="U$2" gate="G$5" pin="PE5"/>
 <label x="147.32" y="157.48" size="1.778" layer="95"/>
@@
 <segment>
 <wire x1="162.56" y1="154.94" x2="127" y2="154.94" width="0.1524" layer="91"/>
-<wire x1="198.12" y1="170.18" x2="162.56" y2="170.18" width="0.1524" layer="91"/>
 <wire x1="162.56" y1="170.18" x2="162.56" y2="154.94" width="0.1524" layer="91"/>
-<pinref part="U$1" gate="G$1" pin="2-TXD"/>
 <pinref part="U$2" gate="G$5" pin="PE4"/>
 <label x="147.32" y="154.94" size="1.778" layer="95"/>
@@
 <segment>
 <wire x1="165.1" y1="147.32" x2="127" y2="147.32" width="0.1524" layer="91"/>
-<wire x1="198.12" y1="149.86" x2="165.1" y2="149.86" width="0.1524" layer="91"/>
 <wire x1="165.1" y1="149.86" x2="165.1" y2="147.32" width="0.1524" layer="91"/>
-<pinref part="U$1" gate="G$1" pin="6-RST_B"/>
 <pinref part="U$2" gate="G$5" pin="PE1"/>
 <label x="147.32" y="147.32" size="1.778" layer="95"/>
@@
 <segment>
 <wire x1="170.18" y1="144.78" x2="170.18" y2="165.1" width="0.1524" layer="91"/>
-<wire x1="170.18" y1="165.1" x2="198.12" y2="165.1" width="0.1524" layer="91"/>
-<pinref part="U$1" gate="G$1" pin="3-GPIO_2"/>
 <wire x1="127" y1="144.78" x2="170.18" y2="144.78" width="0.1524" layer="91"/>
 <pinref part="U$2" gate="G$5" pin="PE0"/>
@@
 <net name="8266_GPIO_0" class="0">
 <segment>
-<wire x1="198.12" y1="154.94" x2="175.26" y2="154.94" width="0.1524" layer="91"/>
 <pinref part="R3" gate="G$1" pin="1"/>
 <wire x1="175.26" y1="154.94" x2="175.26" y2="172.72" width="0.1524" layer="91"/>
-<pinref part="U$1" gate="G$1" pin="5-GPIO_0"/>
 <label x="177.8" y="154.94" size="1.524" layer="95"/>
 </segment>
